File: schematics/carbonATX/CarbonZ80/200x300_64pin_4.kicad_pcb (KiCad board)
At the start: 2 copper layers, 300 x 200 mm, 14 parts

Commit message: placed objects yo
Changed lines of the file:
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@@
 			(psnegative no)
 			(psa4output no)
-			(plot_black_and_white yes)
+			(plot_black_and_white no)
 			(plotinvisibletext no)
 			(sketchpadsonfab no)
@@
 			(crossoutdnponfab yes)
 			(subtractmaskfromsilk no)
-			(outputformat 1)
+			(outputformat 5)
 			(mirror no)
-			(drillshape 1)
+			(drillshape 0)
 			(scaleselection 1)
 			(outputdirectory "")
@@
 	)
 	(gr_rect
+		(start 40 40)
+		(end 325 230)
+		(stroke
+			(width 0.2)
+			(type solid)
+		)
+		(fill no)
+		(layer "F.SilkS")
+	)
+	(gr_rect
