File: schematics/carbonATX/CarbonZ80/CarbonZ80.kicad_pcb (KiCad board)
At the start: 2 copper layers, 300 x 200 mm, 26 parts, among them IC2 CTC-DIP-28, IC3 SIO2-DIP-40, IC4 SIO2-DIP-40, J1 DE9_Socket_MountingHoles, J2 DB25_Socket_MountingHoles, J4 Barrel_Jack_MountingPin, U1 PIO-DIP-40, U2 PIO-DIP-40, U3 PIO-DIP-40, U4 PIO-DIP-40, U5 Z80CPU, U6 YM2149

Commit message: fixed rough layout
Parts:
- removed J2: DB25_Socket_MountingHoles, Connector_Dsub:DSUB-25_Socket_Horizontal_P2.77x2.84mm_EdgePinOffset7.70mm_Housed_MountingHolesOffset9.12mm
- added U7: PIO-DIP-40, Package_DIP:DIP-40_W15.24mm_Socket_LongPads, F.Cu at (289.7, 151.5)
- U6: footprint Package_DIP:DIP-40_W15.24mm_Socket_LongPads -> Package_DIP:DIP-24_W15.24mm_Socket_LongPads
- moved IC2 86.2 mm to (291.4, 121.9)
- moved J1 60.5 mm to (294.0, 44.9)
- moved IC4 46.1 mm to (276.3, 76.7), turned to 90 degrees
- moved U5 40.7 mm to (284.6, 106.5), turned to -90 degrees
- moved U6 32.9 mm to (324.4, 151.5), turned to -90 degrees
- moved IC3 22.3 mm to (221.4, 76.6), turned to 90 degrees
- moved U3 12.8 mm to (98.0, 145.8)
- moved U2 0.20 mm to (136.5, 151.3)
- moved U4 0.16 mm to (56.5, 151.3)

Commit message: updates
Parts:
- added IC1: DMA-DIP-40, Package_DIP:DIP-40_W15.24mm_Socket_LongPads, F.Cu at (324.7, 131.5)
- U6: value YM2149 -> AM9511 (temp)
- moved U6 15.0 mm to (324.4, 166.5)
- moved U7 15.0 mm to (289.7, 166.5)
- moved IC2 10.0 mm to (291.4, 111.9)
- moved U5 10.0 mm to (284.6, 96.5)

Commit message: upd
Parts:
- removed IC3: SIO2-DIP-40, Package_DIP:DIP-40_W15.24mm_Socket_LongPads
- removed U7: PIO-DIP-40, Package_DIP:DIP-40_W15.24mm_Socket_LongPads
- added ?: , Carbonz80_Library:8bISA_64pin, F.Cu at (121.1, 60.2)
- added ?: , Carbonz80_Library:8bISA_64pin, F.Cu at (80.5, 60.2)
- added ?: , Carbonz80_Library:8bISA_64pin, F.Cu at (161.8, 60.2)
- added PIO0: PIO-DIP-40, Package_DIP:DIP-40_W15.24mm_Socket_LongPads, F.Cu at (271.5, 61.4)
- moved DMA0 84.4 mm to (244.3, 157.0), turned to 0 degrees
- moved CPU0 78.5 mm to (211.5, 67.9), turned to 0 degrees
- moved FPU0 72.8 mm to (271.5, 116.5), turned to 0 degrees
- moved SIO0 33.8 mm to (306.5, 61.5), turned to 0 degrees
- moved PIO3 28.1 mm to (86.5, 171.5)
- moved PIO2 20.2 mm to (136.5, 171.5)
- moved PIO4 20.1 mm to (56.5, 171.5)
- moved PIO1 20.0 mm to (181.5, 171.5)
- moved CTC0 15.8 mm to (306.5, 116.5), turned to 0 degrees
- renumbered U5 to CPU0, IC2 to CTC0, IC1 to DMA0, U6 to FPU0, U1 to PIO1, U2 to PIO2, U3 to PIO3, U4 to PIO4, IC4 to SIO0

Commit message: more progress
Parts:
- removed the ? at (108.4, 199.9)
- removed the ? at (121.1, 60.2)
- removed the ? at (80.5, 60.2)
- removed the ? at (161.8, 60.2)
- removed the ? at (128.7, 199.9)
- added RAM0: AS6C4008, PCM_Package_DIP_AKL:DIP-32_W15.24mm_Socket, F.Cu at (304.8, 181.4)
- added RAM1: IDT6116, Package_DIP:DIP-24_W15.24mm_Socket, F.Cu at (271.5, 191.6)
- added ROM0: W27C512, Package_DIP:DIP-28_W15.24mm_Socket, F.Cu at (236.5, 186.5)
- CPU0: value Z80CPU -> Z84C00; footprint Package_DIP:DIP-40_W15.24mm_Socket_LongPads -> Package_DIP:DIP-40_W15.24mm_Socket
- CTC0: value CTC-DIP-28 -> Z84C30; footprint Package_DIP:DIP-28_W15.24mm_Socket_LongPads -> Package_DIP:DIP-28_W15.24mm_Socket
- DMA0: value DMA-DIP-40 -> Z84C10; footprint Package_DIP:DIP-40_W15.24mm_Socket_LongPads -> Package_DIP:DIP-40_W15.24mm_Socket
- FPU0: value AM9511 (temp) -> Am9511A; footprint Package_DIP:DIP-24_W15.24mm_Socket_LongPads -> Package_DIP:DIP-24_W15.24mm_Socket
- PIO0, PIO1, PIO2, PIO3, PIO4: value PIO-DIP-40 -> Z84C20; footprint Package_DIP:DIP-40_W15.24mm_Socket_LongPads -> Package_DIP:DIP-40_W15.24mm_Socket
- SIO0: value SIO2-DIP-40 -> Z84C42; footprint Package_DIP:DIP-40_W15.24mm_Socket_LongPads -> Package_DIP:DIP-40_W15.24mm_Socket
- moved CPU0 104.9 mm to (196.5, 171.8)
- moved DMA0 95.9 mm to (236.3, 61.4)
- moved PIO0 69.6 mm to (236.3, 121.4)
- moved CTC0 55.1 mm to (304.8, 61.4)
- moved SIO0 35.0 mm to (271.5, 61.2)
- moved FPU0 34.6 mm to (271.5, 151.0)
- moved PIO1 30.2 mm to (151.3, 171.5)
- moved PIO2 16.7 mm to (119.8, 171.6)
- moved PIO3 1.77 mm to (88.3, 171.6)
- moved PIO4 0.77 mm to (57.3, 171.6)
Connections:
- FPU0 pad 6: unconnected-(FPU0-IOB7-Pad6) -> (no net)
- FPU0 pad 7: unconnected-(FPU0-IOB6-Pad7) -> (no net)

Commit message: big updates
Parts:
- removed the ? at (141.4, 60.2)
- removed the ? at (60.2, 60.2)
- removed the ? at (100.8, 60.2)
- removed the ? at (182.1, 60.2)
- added BUS0: BUS_SLOT1, CarbonZ80_Library:8bISA_64pin, F.Cu at (182.1, 60.2)
- added BUS1: BUS_SLOT2, CarbonZ80_Library:8bISA_64pin, F.Cu at (141.4, 60.2)
- added BUS2: BUS_SLOT3, CarbonZ80_Library:8bISA_64pin, F.Cu at (100.8, 60.2)
- added BUS3: BUS_SLOT4, CarbonZ80_Library:8bISA_64pin, F.Cu at (60.2, 60.2)
- added DIN0: MINI_DIN_KEYB, CarbonZ80_Library:Mini_DIN_6, F.Cu at (261.6, 34.5)
- added SWT0: RAM_SIZE_SEL, Connector_PinHeader_2.54mm:PinHeader_1x03_P2.54mm_Vertical, F.Cu at (310.0, 174.0)
- COM0: renamed from J1; value DE9_Socket_MountingHoles -> DE9_SOCKET
- FPU0: value Am9511A -> AM9511A
- PWR0: renamed from J4; value Barrel_Jack_MountingPin -> BARREL_JACK_5.5x2.1
- ROM0: value W27C512 -> AT28C64B
- moved FPU0 19.5 mm to (271.4, 131.5)
- moved COM0 4.00 mm to (290.0, 44.9)
- moved PWR0 0.50 mm to (326.5, 44.5)
Connections:
- CPU0 pad 11: unconnected-(CPU0-VCC-Pad11) -> VCC
- CPU0 pad 16: unconnected-(CPU0-~{INT}-Pad16) -> Net-(CPU0-~{INT})
- CPU0 pad 19: unconnected-(CPU0-~{MREQ}-Pad19) -> Net-(CPU0-~{MREQ})
- CPU0 pad 20: unconnected-(CPU0-~{IORQ}-Pad20) -> Net-(CPU0-~{IORQ})
- CPU0 pad 21: unconnected-(CPU0-~{RD}-Pad21) -> Net-(CPU0-~{RD})
- CPU0 pad 22: unconnected-(CPU0-~{WR}-Pad22) -> Net-(CPU0-~{WR})
- CPU0 pad 24: unconnected-(CPU0-~{WAIT}-Pad24) -> Net-(CPU0-~{WAIT})
- CPU0 pad 29: unconnected-(CPU0-GND-Pad29) -> GND
- CTC0 pad 10: unconnected-(CTC0-~{IORQ}-Pad10) -> Net-(CPU0-~{IORQ})
- CTC0 pad 11: unconnected-(CTC0-IEO-Pad11) -> Net-(CTC0-IEO)
- CTC0 pad 12: unconnected-(CTC0-~{INT}-Pad12) -> Net-(CPU0-~{INT})
- CTC0 pad 13: unconnected-(CTC0-IEI-Pad13) -> VCC
- CTC0 pad 14: unconnected-(CTC0-~{M1}-Pad14) -> Net-(CPU0-~{WAIT})
- CTC0 pad 24: unconnected-(CTC0-+5V-Pad24) -> VCC
- CTC0 pad 5: unconnected-(CTC0-GND-Pad5) -> GND
- CTC0 pad 6: unconnected-(CTC0-~{RD}-Pad6) -> Net-(CPU0-~{RD})
- CTC0 pad 8: unconnected-(CTC0-ZC/TO1-Pad8) -> Net-(CTC0-ZC/TO1)
- CTC0 pad 9: unconnected-(CTC0-ZC/TO2-Pad9) -> Net-(CTC0-ZC/TO2)
- DMA0 pad 10: unconnected-(DMA0-~{IORQ}-Pad10) -> Net-(CPU0-~{IORQ})
- DMA0 pad 11: unconnected-(DMA0-VCC-Pad11) -> VCC
- DMA0 pad 12: unconnected-(DMA0-~{MREQ}-Pad12) -> Net-(CPU0-~{MREQ})
- DMA0 pad 25: unconnected-(DMA0-RDY-Pad25) -> Net-(DMA0-RDY)
- DMA0 pad 26: unconnected-(DMA0-~{M1}-Pad26) -> Net-(CPU0-~{WAIT})
- DMA0 pad 30: unconnected-(DMA0-GND-Pad30) -> GND
- DMA0 pad 36: unconnected-(DMA0-IEO-Pad36) -> Net-(DMA0-IEO)
- DMA0 pad 37: unconnected-(DMA0-~{INT/PULSE}-Pad37) -> Net-(CPU0-~{INT})
- DMA0 pad 38: unconnected-(DMA0-IEI-Pad38) -> GND
- DMA0 pad 8: unconnected-(DMA0-~{WR}-Pad8) -> Net-(CPU0-~{WR})
- DMA0 pad 9: unconnected-(DMA0-~{RD}-Pad9) -> Net-(CPU0-~{RD})
- FPU0 pad 1: unconnected-(FPU0-VSS-Pad1) -> GND
- FPU0 pad 10: unconnected-(FPU0-DB2-Pad10) -> Net-(FPU0-DB2)
- FPU0 pad 11: unconnected-(FPU0-DB3-Pad11) -> Net-(FPU0-DB3)
- FPU0 pad 12: unconnected-(FPU0-DB4-Pad12) -> Net-(FPU0-DB4)
- FPU0 pad 13: unconnected-(FPU0-DB5-Pad13) -> Net-(FPU0-DB5)
- FPU0 pad 14: unconnected-(FPU0-DB6-Pad14) -> Net-(FPU0-DB6)
- FPU0 pad 15: unconnected-(FPU0-DB7-Pad15) -> Net-(FPU0-DB7)
- FPU0 pad 2: unconnected-(FPU0-VCC-Pad2) -> VCC
- FPU0 pad 8: unconnected-(FPU0-DB0-Pad8) -> Net-(FPU0-DB0)
- FPU0 pad 9: unconnected-(FPU0-DB1-Pad9) -> Net-(FPU0-DB1)
- PIO0 pad 10: unconnected-(PIO0-PA4-Pad10) -> Net-(FPU0-DB4)
- PIO0 pad 11: unconnected-(PIO0-GND-Pad11) -> GND
- PIO0 pad 12: unconnected-(PIO0-PA3-Pad12) -> Net-(FPU0-DB3)
- PIO0 pad 13: unconnected-(PIO0-PA2-Pad13) -> Net-(FPU0-DB2)
- PIO0 pad 14: unconnected-(PIO0-PA1-Pad14) -> Net-(FPU0-DB1)
- PIO0 pad 15: unconnected-(PIO0-PA0-Pad15) -> Net-(FPU0-DB0)
- PIO0 pad 22: unconnected-(PIO0-IEO-Pad22) -> Net-(PIO0-IEO)
- PIO0 pad 23: unconnected-(PIO0-~{INT}-Pad23) -> Net-(CPU0-~{INT})
- PIO0 pad 24: unconnected-(PIO0-IEI-Pad24) -> Net-(DMA0-IEO)
- PIO0 pad 26: unconnected-(PIO0-VCC-Pad26) -> VCC
- PIO0 pad 7: unconnected-(PIO0-PA7-Pad7) -> Net-(FPU0-DB7)
- PIO0 pad 8: unconnected-(PIO0-PA6-Pad8) -> Net-(FPU0-DB6)
- PIO0 pad 9: unconnected-(PIO0-PA5-Pad9) -> Net-(FPU0-DB5)
- PIO1 pad 11: unconnected-(PIO1-GND-Pad11) -> GND
- PIO1 pad 22: unconnected-(PIO1-IEO-Pad22) -> Net-(PIO1-IEO)
- PIO1 pad 23: unconnected-(PIO1-~{INT}-Pad23) -> Net-(CPU0-~{INT})
- PIO1 pad 24: unconnected-(PIO1-IEI-Pad24) -> Net-(PIO0-IEO)
- PIO1 pad 26: unconnected-(PIO1-VCC-Pad26) -> VCC
- PIO2 pad 11: unconnected-(PIO2-GND-Pad11) -> GND
- PIO2 pad 22: unconnected-(PIO2-IEO-Pad22) -> GND
- PIO2 pad 23: unconnected-(PIO2-~{INT}-Pad23) -> Net-(CPU0-~{INT})
- PIO2 pad 24: unconnected-(PIO2-IEI-Pad24) -> Net-(PIO1-IEO)
- PIO2 pad 26: unconnected-(PIO2-VCC-Pad26) -> VCC
- PIO3 pad 11: unconnected-(PIO3-GND-Pad11) -> GND
- PIO3 pad 22: unconnected-(PIO3-IEO-Pad22) -> Net-(PIO3-IEO)
- PIO3 pad 23: unconnected-(PIO3-~{INT}-Pad23) -> Net-(CPU0-~{INT})
- PIO3 pad 24: unconnected-(PIO3-IEI-Pad24) -> GND
- PIO3 pad 26: unconnected-(PIO3-VCC-Pad26) -> VCC
- PIO4 pad 11: unconnected-(PIO4-GND-Pad11) -> GND
- PIO4 pad 23: unconnected-(PIO4-~{INT}-Pad23) -> Net-(CPU0-~{INT})
- PIO4 pad 24: unconnected-(PIO4-IEI-Pad24) -> Net-(PIO3-IEO)
- PIO4 pad 26: unconnected-(PIO4-VCC-Pad26) -> VCC
- RAM0 pad 16: unconnected-(RAM0-VSS-Pad16) -> GND
- RAM0 pad 22: unconnected-(RAM0-CE#-Pad22) -> Net-(RAM0-CE#)
- RAM0 pad 24: unconnected-(RAM0-OE#-Pad24) -> Net-(CPU0-~{RD})
- RAM0 pad 29: unconnected-(RAM0-WE#-Pad29) -> Net-(CPU0-~{WR})
- RAM0 pad 32: unconnected-(RAM0-VCC-Pad32) -> VCC
- RAM1 pad 12: unconnected-(RAM1-GND-Pad12) -> GND
- RAM1 pad 18: unconnected-(RAM1-~{CS}-Pad18) -> Net-(RAM1-~{CS})
- RAM1 pad 20: unconnected-(RAM1-~{OE}-Pad20) -> Net-(CPU0-~{RD})
- RAM1 pad 21: unconnected-(RAM1-~{WE}-Pad21) -> Net-(CPU0-~{WR})
- RAM1 pad 24: unconnected-(RAM1-VCC-Pad24) -> VCC
- ROM0 pad 14: unconnected-(ROM0-GND-Pad14) -> GND
- ROM0 pad 22: unconnected-(ROM0-~{OE/Vpp}-Pad22) -> Net-(CPU0-~{RD})
- ROM0 pad 28: unconnected-(ROM0-VCC-Pad28) -> VCC
- SIO0 pad 13: unconnected-(SIO0-~{RXCA}-Pad13) -> Net-(CTC0-ZC/TO2)
- SIO0 pad 14: unconnected-(SIO0-~{TXCA}-Pad14) -> Net-(CTC0-ZC/TO2)
- SIO0 pad 27: unconnected-(SIO0-~{TXCB}-Pad27) -> Net-(CTC0-ZC/TO1)
- SIO0 pad 28: unconnected-(SIO0-~{RXCB}-Pad28) -> Net-(CTC0-ZC/TO1)
- SIO0 pad 30: unconnected-(SIO0-~{W}/~{RDYB}-Pad30) -> Net-(DMA0-RDY)
- SIO0 pad 31: unconnected-(SIO0-GND-Pad31) -> GND
- SIO0 pad 5: unconnected-(SIO0-~{INT}-Pad5) -> Net-(CPU0-~{INT})
- SIO0 pad 6: unconnected-(SIO0-IEI-Pad6) -> Net-(CTC0-IEO)
- SIO0 pad 7: unconnected-(SIO0-IEO-Pad7) -> GND
- SIO0 pad 9: unconnected-(SIO0-+5V-Pad9) -> VCC
