File: schematics/carbonATX/CarbonZ80/CarbonZ80.kicad_sch (KiCad schematic)
At the start: 13 parts, among them IC2 CTC-DIP-28, IC3 SIO2-DIP-40, IC4 SIO2-DIP-40, J1 DE9_Socket_MountingHoles, J2 DB25_Socket_MountingHoles, J3 Mini-DIN-6, J4 Barrel_Jack_MountingPin, U1 PIO-DIP-40, U2 PIO-DIP-40, U3 PIO-DIP-40, U4 PIO-DIP-40, U5 Z80CPU, U6 YM2149

Commit message: fixed rough layout
Parts:
- removed J2: DB25_Socket_MountingHoles, Connector_Dsub:DSUB-25_Socket_Horizontal_P2.77x2.84mm_EdgePinOffset7.70mm_Housed_MountingHolesOffset9.12mm, symbol Connector:DB25_Socket_MountingHoles
- added U7: PIO-DIP-40, Package_DIP:DIP-40_W15.24mm_Socket_LongPads, symbol Zilog_Z80_Peripherals:PIO-DIP-40
- U6: footprint Package_DIP:DIP-40_W15.24mm_Socket_LongPads -> Package_DIP:DIP-24_W15.24mm_Socket_LongPads
Other:
- moved on the sheet: U6
Changed lines of the file:
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@@
 	(title_block
 		(title "Carbon Z80 - 4x Slots & Mode 2 Ints")
-		(date "2025-02-25")
-		(rev "0")
+		(date "2025-02-27")
+		(rev "1")
 		(company "Jules Carboni")
 	)
@@
 	(symbol
 		(lib_id "Zilog_Z80_Peripherals:PIO-DIP-40")
+		(at 120.65 179.07 0)
+		(unit 1)
+		(exclude_from_sim no)
+		(in_bom yes)
+		(on_board yes)
+		(dnp no)
+		(fields_autoplaced yes)
+		(property "Reference" "U7"
+			(at 132.9533 173.99 0)
+			(effects
+				(font
+					(size 1.27 1.27)
+				)
+				(justify left)
+			)
+		)
+		(property "Value" "PIO-DIP-40"
+			(at 132.9533 176.53 0)
+			(effects
+				(font
+					(size 1.27 1.27)
+				)
+				(justify left)
+			)
+		)
+		(property "Footprint" "Package_DIP:DIP-40_W15.24mm_Socket_LongPads"
+			(at 130.81 245.11 0)
+			(effects
+				(font
+					(size 1.27 1.27)
+				)
+				(hide yes)
+			)
+		)
+		(property "Datasheet" "https://www.zilog.com/appnotes_download.php?FromPage=DirectLink&dn=PS0180&ft=Product%20Specification%20(Data%20Sheet)%20%20&f=YUhSMGNEb3ZMM2QzZHk1NmFXeHZaeTVqYjIwdlpHOWpjeTk2T0RBdmNITXdNVGd3TG5Ca1pnPT0="
+			(at 119.38 219.71 0)
+			(effects
+				(font
+					(size 1.27 1.27)
+				)
+				(hide yes)
+			)
+		)
+		(property "Description" "ZILOG PIO DIP-40 Z84C20 Z8420"
+			(at 120.65 179.07 0)
+			(effects
+				(font
+					(size 1.27 1.27)
+				)
+				(hide yes)
+			)
+		)
+		(pin "17"
+		)
+		(pin "23"
+		)
+		(pin "6"
+		)
+		(pin "14"
+		)
+		(pin "27"
+		)
+		(pin "28"
+		)
+		(pin "24"
+		)
+		(pin "21"
+		)
+		(pin "16"
+		)
+		(pin "19"
+		)
+		(pin "25"
+		)
+		(pin "5"
+		)
+		(pin "4"
+		)
+		(pin "35"
+		)
+		(pin "38"
+		)
+		(pin "22"
+		)
+		(pin "11"
+		)
+		(pin "13"
+		)
+		(pin "10"
+		)
+		(pin "7"
+		)
+		(pin "30"
+		)
+		(pin "26"
+		)
+		(pin "15"
+		)
+		(pin "2"
+		)
+		(pin "3"
+		)
+		(pin "12"
+		)
+		(pin "8"
+		)
+		(pin "31"
+		)
+		(pin "20"
+		)
+		(pin "1"
+		)
+		(pin "37"
+		)
+		(pin "18"
+		)
+		(pin "29"
+		)
+		(pin "32"
+		)
+		(pin "33"
+		)
+		(pin "39"
+		)
+		(pin "34"
+		)
+		(pin "36"
+		)
+		(pin "9"
+		)
+		(pin "40"
+		)
+		(instances
+			(project "CarbonZ80"
+				(path "/6e4cebc6-dd58-4879-8795-195abcf058ff"
+					(reference "U7")
+					(unit 1)
+				)
+			)
+		)
+	)
+	(symbol
+		(lib_id "Zilog_Z80_Peripherals:PIO-DIP-40")
 		(at 332.74 179.07 0)
 		(unit 1)
@@
 	)
 	(symbol
-		(lib_id "Connector:DB25_Socket_MountingHoles")
-		(at 388.62 203.2 0)
-		(unit 1)
-		(exclude_from_sim no)
-		(in_bom yes)
-		(on_board yes)
-		(dnp no)
-		(fields_autoplaced yes)
-		(property "Reference" "J2"
-			(at 393.7 201.9299 0)
-			(effects
-				(font
-					(size 1.27 1.27)
-				)
-				(justify left)
-			)
-		)
-		(property "Value" "DB25_Socket_MountingHoles"
-			(at 393.7 204.4699 0)
-			(effects
-				(font
-					(size 1.27 1.27)
-				)
-				(justify left)
-			)
-		)
-		(property "Footprint" "Connector_Dsub:DSUB-25_Socket_Horizontal_P2.77x2.84mm_EdgePinOffset7.70mm_Housed_MountingHolesOffset9.12mm"
-			(at 388.62 203.2 0)
-			(effects
-				(font
-					(size 1.27 1.27)
-				)
-				(hide yes)
-			)
-		)
-		(property "Datasheet" "~"
-			(at 388.62 203.2 0)
-			(effects
-				(font
-					(size 1.27 1.27)
-				)
-				(hide yes)
-			)
-		)
-		(property "Description" "25-pin D-SUB connector, socket (female), Mounting Hole"
-			(at 388.62 203.2 0)
-			(effects
-				(font
-					(size 1.27 1.27)
-				)
-				(hide yes)
-			)
-		)
-		(pin "17"
-		)
-		(pin "9"
-		)
-		(pin "22"
-		)
-		(pin "10"
-		)
-		(pin "5"
-		)
-		(pin "2"
-		)
-		(pin "15"
-		)
-		(pin "3"
-		)
-		(pin "16"
-		)
-		(pin "4"
-		)
-		(pin "6"
-		)
-		(pin "7"
-		)
-		(pin "20"
-		)
-		(pin "14"
-		)
-		(pin "18"
-		)
-		(pin "19"
-		)
-		(pin "1"
-		)
-		(pin "8"
-		)
-		(pin "21"
-		)
-		(pin "23"
-		)
-		(pin "11"
-		)
-		(pin "24"
-		)
-		(pin "25"
-		)
-		(pin "13"
-		)
-		(pin "12"
-		)
-		(pin "0"
-		)
-		(instances
-			(project ""
-				(path "/6e4cebc6-dd58-4879-8795-195abcf058ff"
-					(reference "J2")
-					(unit 1)
-				)
-			)
-		)
-	)
-	(symbol
 		(lib_id "Connector:Barrel_Jack_MountingPin")
 		(at 30.48 30.48 0)
@@
 	(symbol
 		(lib_id "Audio:YM2149")
-		(at 91.44 207.01 0)
+		(at 71.12 207.01 0)
 		(unit 1)
 		(exclude_from_sim no)
@@
 		(fields_autoplaced yes)
 		(property "Reference" "U6"
-			(at 93.5833 173.99 0)
+			(at 73.2633 173.99 0)
 			(effects
 				(font
@@
 		)
 		(property "Value" "YM2149"
-			(at 93.5833 176.53 0)
-			(effects
-				(font
-					(size 1.27 1.27)
-				)
-				(justify left)
-			)
-		)
-		(property "Footprint" "Package_DIP:DIP-40_W15.24mm_Socket_LongPads"
-			(at 107.95 242.57 0)
+			(at 73.2633 176.53 0)
+			(effects
+				(font
+					(size 1.27 1.27)
+				)
+				(justify left)
+			)
+		)
+		(property "Footprint" "Package_DIP:DIP-24_W15.24mm_Socket_LongPads"
+			(at 87.63 242.57 0)
 			(effects
 				(font
@@
 		)
 		(property "Datasheet" "http://www.ym2149.com/ym2149.pdf"
-			(at 91.44 207.01 0)
+			(at 71.12 207.01 0)
 			(effects
 				(font
@@
 		)
 		(property "Description" "Software-Controlled Sound Generator, DIP-40"
-			(at 91.44 207.01 0)
-			(effects
-				(font
+			(at 71.12 207.01 0)
+			(effects
+				(font

Commit message: more updates
Parts:
- added IC1: DMA-DIP-40, Package_DIP:DIP-40_W15.24mm_Socket_LongPads, symbol Zilog_Z80_Peripherals:DMA-DIP-40
- U6: value YM2149 -> AM9511 (temp)
Connections:
- no-connect marks 0 -> 1
Other:
- moved on the sheet: IC2, IC3, IC4, J1, J3, U1, U2, U3, U4, U5, U6, U7

Commit message: upd
Parts:
- removed IC3: SIO2-DIP-40, Package_DIP:DIP-40_W15.24mm_Socket_LongPads, symbol Zilog_Z80_Peripherals:SIO2-DIP-40
- removed U7: PIO-DIP-40, Package_DIP:DIP-40_W15.24mm_Socket_LongPads, symbol Zilog_Z80_Peripherals:PIO-DIP-40
- added PIO0: PIO-DIP-40, Package_DIP:DIP-40_W15.24mm_Socket_LongPads, symbol Zilog_Z80_Peripherals:PIO-DIP-40
- renumbered U5 to CPU0, IC2 to CTC0, IC1 to DMA0, U6 to FPU0, U1 to PIO1, U2 to PIO2, U3 to PIO3, U4 to PIO4, IC4 to SIO0
Other:
- moved on the sheet: CTC0, FPU0

Commit message: more progress
Parts:
- removed FPU0: AM9511 (temp), Package_DIP:DIP-24_W15.24mm_Socket_LongPads, symbol Audio:YM2149
- added FPU0: Am9511A, Package_DIP:DIP-24_W15.24mm_Socket, symbol CarbonZ80_Library:Am9511
- added RAM0: AS6C4008, PCM_Package_DIP_AKL:DIP-32_W15.24mm_Socket, symbol Memory_RAM:AS6C4008-55PCN
- added RAM1: IDT6116, Package_DIP:DIP-24_W15.24mm_Socket, symbol CarbonZ80_Library:IDT6116
- added ROM0: W27C512, Package_DIP:DIP-28_W15.24mm_Socket, symbol 8Bit_Chips:W27C512
- CPU0: value Z80CPU -> Z84C00; footprint Package_DIP:DIP-40_W15.24mm_Socket_LongPads -> Package_DIP:DIP-40_W15.24mm_Socket
- CTC0: value CTC-DIP-28 -> Z84C30; footprint Package_DIP:DIP-28_W15.24mm_Socket_LongPads -> Package_DIP:DIP-28_W15.24mm_Socket
- DMA0: value DMA-DIP-40 -> Z84C10; footprint Package_DIP:DIP-40_W15.24mm_Socket_LongPads -> Package_DIP:DIP-40_W15.24mm_Socket
- PIO0, PIO1, PIO2, PIO3, PIO4: value PIO-DIP-40 -> Z84C20; footprint Package_DIP:DIP-40_W15.24mm_Socket_LongPads -> Package_DIP:DIP-40_W15.24mm_Socket
- SIO0: value SIO2-DIP-40 -> Z84C42; footprint Package_DIP:DIP-40_W15.24mm_Socket_LongPads -> Package_DIP:DIP-40_W15.24mm_Socket
Connections:
- no-connect marks 1 -> 0
Other:
- moved on the sheet: CPU0, PIO0, PIO1, PIO2, PIO3, PIO4

Commit message: big updates
Parts:
- added BUS0: BUS_SLOT1, CarbonZ80_Library:8bISA_64pin, symbol CarbonZ80_Library:Bus_ISA_8bit_64pin
- added BUS1: BUS_SLOT2, CarbonZ80_Library:8bISA_64pin, symbol CarbonZ80_Library:Bus_ISA_8bit_64pin
- added BUS2: BUS_SLOT3, CarbonZ80_Library:8bISA_64pin, symbol CarbonZ80_Library:Bus_ISA_8bit_64pin
- added BUS3: BUS_SLOT4, CarbonZ80_Library:8bISA_64pin, symbol CarbonZ80_Library:Bus_ISA_8bit_64pin
- added SWT0: RAM_SIZE_SEL, Connector_PinHeader_2.54mm:PinHeader_1x03_P2.54mm_Vertical, symbol PCM_SL_Pin_Headers:PINHD_1x3_Male
- COM0: renamed from J1; value DE9_Socket_MountingHoles -> DE9_SOCKET
- DIN0: renamed from J3; value Mini-DIN-6 -> MINI_DIN_KEYB; footprint (none) -> CarbonZ80_Library:Mini_DIN_6
- FPU0: value Am9511A -> AM9511A
- PWR0: renamed from J4; value Barrel_Jack_MountingPin -> BARREL_JACK_5.5x2.1
- ROM0: value W27C512 -> AT28C64B
Connections:
- net VCC: now reaches CPU0.11 (VCC)
- net VCC: now also CTC0.13 (IEI), CTC0.24 (+5V), DMA0.11 (VCC), FPU0.2 (VCC), PIO0.26 (VCC), PIO1.26 (VCC), PIO2.26 (VCC), PIO3.26 (VCC), PIO4.26 (VCC), RAM0.32 (VCC), RAM1.24 (VCC), ROM0.28 (VCC), SIO0.9 (+5V)
- net at CPU0.16 (~{INT}): now also CTC0.12 (~{INT}), DMA0.37 (~{INT/PULSE}), PIO0.23 (~{INT}), PIO1.23 (~{INT}), PIO2.23 (~{INT}), PIO3.23 (~{INT}), PIO4.23 (~{INT}), SIO0.5 (~{INT})
- net at CPU0.19 (~{MREQ}): now also DMA0.12 (~{MREQ})
- net at CPU0.20 (~{IORQ}): now also CTC0.10 (~{IORQ}), DMA0.10 (~{IORQ})
- net at CPU0.21 (~{RD}): now also CTC0.6 (~{RD}), DMA0.9 (~{RD}), RAM0.24 (OE#), RAM1.20 (~{OE}), ROM0.22 (~{OE/Vpp})
- net at CPU0.22 (~{WR}): now also DMA0.8 (~{WR}), RAM0.29 (WE#), RAM1.21 (~{WE})
- net at CPU0.24 (~{WAIT}): now also CTC0.14 (~{M1}), DMA0.26 (~{M1})
- net GND: now reaches CPU0.29 (GND)
- net GND: now also CTC0.5 (GND), DMA0.30 (GND), DMA0.38 (IEI), FPU0.1 (VSS), PIO0.11 (GND), PIO1.11 (GND), PIO2.11 (GND), PIO2.22 (IEO), PIO3.11 (GND), PIO3.24 (IEI), PIO4.11 (GND), RAM0.16 (VSS), RAM1.12 (GND), ROM0.14 (GND), SIO0.31 (GND), SIO0.7 (IEO)
- net at FPU0.10 (DB2): now also PIO0.13 (PA2)
- net at FPU0.11 (DB3): now also PIO0.12 (PA3)
- net at FPU0.12 (DB4): now also PIO0.10 (PA4)
- net at FPU0.13 (DB5): now also PIO0.9 (PA5)
- net at FPU0.14 (DB6): now also PIO0.8 (PA6)
- net at FPU0.15 (DB7): now also PIO0.7 (PA7)
- net at FPU0.8 (DB0): now also PIO0.15 (PA0)
- net at FPU0.9 (DB1): now also PIO0.14 (PA1)
- net at PIO4.24 (IEI): now also PIO3.22 (IEO)
- net at DMA0.25 (RDY): now also SIO0.30 (~{W}/~{RDYB})
- net at DMA0.36 (IEO): now also PIO0.24 (IEI)
- net at SIO0.13 (~{RXCA}): now also CTC0.9 (ZC/TO2), SIO0.14 (~{TXCA})
- net at SIO0.27 (~{TXCB}): now also CTC0.8 (ZC/TO1), SIO0.28 (~{RXCB})
- net at SIO0.6 (IEI): now also CTC0.11 (IEO)
- net at PIO1.22 (IEO): now also PIO2.24 (IEI)
- net at PIO1.24 (IEI): now also PIO0.22 (IEO)
- net at RAM1.18 (~{CS}): now also SWT0.1
- net at RAM0.22 (CE#): now also SWT0.3
- no-connect marks 0 -> 47
Other:
- moved on the sheet: FPU0, PIO0, PIO1, PIO2, PIO3, PIO4, SIO0

Commit message: sch
Parts:
- added C1, C2, C9: 1uF, Capacitor_THT:CP_Radial_D5.0mm_P2.50mm, symbol Clock_module-rescue:CP-Device
- added C3: 0.01uF, Capacitor_THT:C_Disc_D3.0mm_W2.0mm_P2.50mm, symbol Device:C
- added C4, C5, C6, C7, C8: 0.1uF, Capacitor_THT:C_Disc_D3.0mm_W2.0mm_P2.50mm, symbol Device:C
- added D2, D3, D5: RED, LED_THT:LED_D5.0mm, symbol Device:LED
- added R1, R15, R2, R4, R6: 100K, Resistor_THT:R_Axial_DIN0207_L6.3mm_D2.5mm_P7.62mm_Horizontal, symbol Device:R
- added R11, R12, R14: 220, Resistor_THT:R_Axial_DIN0207_L6.3mm_D2.5mm_P7.62mm_Horizontal, symbol Device:R
- added R3, R8, R9: 1K, Resistor_THT:R_Axial_DIN0207_L6.3mm_D2.5mm_P7.62mm_Horizontal, symbol Device:R
- added R5, R7: 10K, Resistor_THT:R_Axial_DIN0207_L6.3mm_D2.5mm_P7.62mm_Horizontal, symbol Device:R
- added RV1: 1M, Potentiometer_THT:Potentiometer_Piher_PT-10-V10_Vertical, symbol Clock_module-rescue:R_POT-Device
- added SW1: Mode, Button_Switch_THT:SW_PUSH_6mm, symbol Switch:SW_Push
- added SW2: Step, Button_Switch_THT:SW_PUSH_6mm, symbol Switch:SW_Push
- added U1: 74LS74, symbol 74xx:74LS74
- added U10, U11, U12: NE555P, Package_DIP:DIP-8_W7.62mm, symbol Timer:NE555P
- added U2: 74LS157, symbol 74xx:74LS157
- added U4: 74LS04, Package_DIP:DIP-14_W7.62mm_Socket, symbol 74xx:74LS04
- added U5: 74LS32, Package_DIP:DIP-14_W7.62mm_Socket, symbol 74xx:74LS32
- added U6: 74LS08, Package_DIP:DIP-14_W7.62mm_Socket, symbol 74xx:74LS08
Connections:
- net GND: now also DIN0.3, PWR0.2, SIO0.18 (~{CTSA}), SIO0.19 (~{DCDA}), SIO0.22 (~{DCDB}), SIO0.23 (~{CTSB}), C1.2, C2.2, C3.2, C4.2, C5.2, C6.2, C7.2, C8.2, R11.2, R12.2, R14.2, R15.2, R5.2, SW2.1, U10.1 (GND), U11.1 (GND), U12.1 (GND), U2.8 (GND), U4.7 (GND), U5.7 (GND), U6.7 (GND)
- net VCC: now also DIN0.4, PWR0.1, C3.1, C5.1, R1.1, R3.1, R6.1, R7.1, R8.1, R9.1, U1.1 (~{R}), U1.4 (~{S}), U10.4 (R), U10.8 (VCC), U11.4 (R), U11.8 (VCC), U12.8 (VCC), U2.16 (VCC), U4.14 (VCC), U5.14 (VCC), U6.14 (VCC)
- net at CPU0.16 (~{INT}), CTC0.12 (~{INT}), DMA0.37 (~{INT/PULSE})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: now also DMA0.36 (IEO), PIO0.24 (IEI)
- net at DMA0.25 (RDY): now also SIO0.10 (~{W}/~{RDYA}); no longer SIO0.30 (~{W}/~{RDYB})
- net at SIO0.29 (RXDB): now also DIN0.1
- net at DIN0.5: now also SIO0.28 (~{RXCB})
- new net: R5.1, R7.2, SW1.2, U12.2 (TR), U12.6 (THR)
- new net: D3.1 (K), R12.1
- new net: C6.1, U12.5 (CV)
- new net: C2.1, R4.2, SW1.1
- new net: R4.1, R8.2, U12.7 (DIS)
- new net: C9.1, R3.2, U12.4 (R)
- new net: C1.1, RV1.2, U10.2 (TR), U10.6 (THR)
- new net: C4.1, U10.5 (CV)
- new net: R1.2, R2.1, U10.7 (DIS)
- new net: R2.2, RV1.1
- new net: R6.2, SW2.2, U11.2 (TR)
- new net: C8.1, U11.5 (CV)
- new net: C7.1, R9.2, U11.6 (THR), U11.7 (DIS)
- new net: U5.1, U6.3
- new net: U5.2, U6.6
- new net: U4.4, U6.10
- new net: U5.3, U6.9
- new net: D2.1 (K), R11.1
- new net: D5.1 (K), R14.1
- new net: U1.2 (D), U1.6 (~{Q})
- new net CLK: D5.2 (A), U4.5, U6.8
- new net HLT: R15.1, U4.3
- new net MODE: D3.2 (A), U12.3 (Q), U4.1, U6.1
- new net SINGLE: U11.3 (Q), U6.5
- new net VARIABLE: U10.3 (Q), U6.2
- new net ~{BRK}: C9.2
- new net ~{CLK_HALF}: U1.5 (Q)
- new net ~{CLK}: U1.3 (C), U4.6
- new net ~{MODE}: D2.2 (A), U4.2, U6.4
- now unconnected: CTC0.8 (ZC/TO1), SIO0.27 (~{TXCB})
- no-connect marks 47 -> 56
Other:
- note added: "Check the 0.1uF on the pin5->gnd connection"
- moved on the sheet: COM0, PIO1, PIO2, PIO3, PIO4, PWR0, RAM1, SWT0

Commit message: started new rc2014 design
Parts:
- removed U1: 74LS74, symbol 74xx:74LS74
Other:
- moved on the sheet: U2
