File: schematics/carbonATX/CarbonZ80/CarbonR80.kicad_sch (KiCad schematic)
At the start: 30 parts, among them J1 ATX-24, J11 Bus_Z80_RC2014_ENH, SW1 SW_RESET, SW2 SW_POWER, U1 74LS14

Commit message: small chg
Parts:
- added D2, D3, D4, D5: LED_POWER, LED_THT:LED_D5.0mm, symbol PCM_SL_Devices:LED
- added R4, R5, R8: Resistor, Resistor_THT:R_Axial_DIN0207_L6.3mm_D2.5mm_P10.16mm_Horizontal, symbol PCM_SL_Resistors:Resistor
- C10, C7, C8, C9: value 1mF_16V -> 1mF_50V
Connections:
- net +12V: now also R1.2
- net +3.3V: now also R4.2
- net +5V: no longer R1.2
- net -12V: now also R5.2
- net GND: now also SW1.2, D2.2, D3.2, D4.2, D5.2; no longer SW1.1
- net RESET: now also R3.1, SW1.1; no longer R2.1, R3.2, SW1.2
- net NMI: now reaches J1.8 (PWR_OK)
- net NMI: now also R3.2; no longer R3.1
- net +5VSB: now reaches J1.9 (+5VSB), R6.2
- net +5VSB: now also R8.2
- new net: D3.1, R4.1
- new net: D4.1, R5.1
- new net: D5.1, R8.1
- new net: D2.1, R2.1
Other:
- note added: "Power LED indicators."
- note added: "Power switch, NMI control, and circuit protection. Assuming clean ATX compliant power signals."
- note removed: "Reset button and Power LED."
- note removed: "is reset circuit active high or low"
- note removed: "power ok nmi interrupt"
- moved on the sheet: +12V, +3.3V, +5V, C1, C11, COM0, D1, DIN0, F1, F2, F3, F4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
